Commit message: Added heat bed visualization

File: src/incubator_description/urdf/incubator_form.xacro (robot description, xacro)
@@ -24,17 +24,4 @@
     <xacro:macro name="thermometer" params="num">
         <link name="t${num}">
-            <visual>
-                <geometry>
-                    <sphere radius="0.0254"/>
-                </geometry>
-                <origin xyz="0 0 ${side_height/2.0}"/>
-                <material name="black"/>
-            </visual>
-            <collision>
-                <geometry>
-                    <sphere radius="0.0254"/>
-                </geometry>
-                <origin xyz="0 0 ${side_height/2.0}"/>
-            </collision>
         </link>
     </xacro:macro>
@@ -47,4 +34,5 @@
     <xacro:thermometer num="2"/>
     <xacro:thermometer num="3"/>
+    <link name="heat_bed" />
     <link name="floor">
         <visual>
@@ -90,15 +78,20 @@
         <parent link="right_wall"/>
         <child link="t1"/>
-        <origin xyz="-${side_depth/2.0+0.0254} 0 0" rpy="0 0 0"/>
+        <origin xyz="-${side_depth/2.0+0.0254} 0 ${side_height/2.0}" rpy="0 0 0"/>
     </joint>
     <joint name="front_wall_t2" type="fixed">
         <parent link="front_wall"/>
         <child link="t2"/>
-        <origin xyz="0 -${side_depth/2.0+0.0254} 0" rpy="0 0 0"/>
+        <origin xyz="0 -${side_depth/2.0+0.0254} ${side_height/2.0}" rpy="0 0 0"/>
     </joint>
     <joint name="front_wall_t3" type="fixed">
         <parent link="front_wall"/>
         <child link="t3"/>
-        <origin xyz="0 ${side_depth/2.0+0.0254} 0" rpy="0 0 0"/>
+        <origin xyz="0 ${side_depth/2.0+0.0254} ${side_height/2.0}" rpy="0 0 0"/>
+    </joint>
+    <joint name="floor_heat_bed" type="fixed">
+        <parent link="floor"/>
+        <child link="heat_bed"/>
+        <origin xyz="0 0 ${side_depth/2.0}"/>
     </joint>
 </robot>

Commit message: Updated urdf to better match actual hardware

File: src/incubator_description/urdf/incubator_form.xacro (robot description, xacro)
@@ -75,8 +75,8 @@
         <origin xyz="0 0 0" rpy="0 0 0" />
     </joint>
-    <joint name="right_wall_t1" type="fixed">
-        <parent link="right_wall"/>
+    <joint name="left_wall_t1" type="fixed">
+        <parent link="left_wall"/>
         <child link="t1"/>
-        <origin xyz="-${side_depth/2.0+0.0254} 0 ${side_height/2.0}" rpy="0 0 0"/>
+        <origin xyz="${side_depth/2.0+0.0254} 0 ${side_height/2.0}" rpy="0 0 0"/>
     </joint>
     <joint name="front_wall_t2" type="fixed">
@@ -93,5 +93,5 @@
         <parent link="floor"/>
         <child link="heat_bed"/>
-        <origin xyz="0 0 ${side_depth/2.0}"/>
+        <origin xyz="0 0 ${side_depth+0.01}"/>
     </joint>
 </robot>
